File: projects/HTVentilation/HTVC_NOPWM.sch (EAGLE design)
At the start: 6 parts

Commit message: new items in the lib + new 4 layer board
Parts:
- removed +12V, +12V1, AGND, AGND9, PAD1, PAD2: (no value), wirepad:3,17/1,3
- added C1: 0.33uF, rcl:CPOL-USE2.5-6
- added C2: 0.1uF, rcl:CPOL-USE2.5-6
- added IC1: 7805T, linear:7805T
- added JP1: (no value), SparkFun-Connectors:M03POLAR
Connections:
- removed net T1: PAD1.P
- removed net T2: PAD2.P
- new net +5V: C2.+, IC1.VO
- net AGND: now also C1.-, C2.-, IC1.GND, JP1.2; no longer AGND.P, AGND9.P, PAD2.P
- net VCC: now also C1.+, IC1.VI, JP1.3; no longer +12V.P, +12V1.P, PAD1.P
