File: projects/HTVentilation/HTVC8038_Display_v12.sch (EAGLE design)
At the start: 6 parts

Commit message: cleanup
Parts:
- removed +12V, AGND, PAD1, PAD2: (no value), wirepad:3,17/1,3
Connections:
- removed net FILT_IN: PAD1.P
- removed net T1: PAD1.P
- removed net T2: PAD2.P
- net AGND: no longer AGND.P, PAD2.P
- net VCC: no longer +12V.P, PAD1.P
